Commit message: add folder

File: robot_description/urdf/robot.urdf.xacro (robot description, xacro)
@@ -1,4 +1,4 @@
 <?xml version="1.0"?>
-<robot name ="robotTRUNG" xmlns:xacro="http://ros.org/wiki/xacro" >
+<robot name ="alphabot" xmlns:xacro="http://ros.org/wiki/xacro" >
     <xacro:arg name="is_sim" default="true"/>
     <xacro:include filename="robot_core.xacro" />

File: robot_description/urdf/robot_core.xacro (robot description, xacro)
@@ -1,20 +1,19 @@
 <?xml version="1.0" encoding="utf-8"?>
 <robot xmlns:xacro="http://ros.org/wiki/xacro">
-  <link name="base_footprint"/>
   <link
     name="base_link">
     <inertial>
       <origin
-        xyz="-0.0218638387317892 -0.00507304700544385 0.0654073746420509"
-        rpy="0 0 0" />
-      <mass
-        value="1.60320284644643" />
-      <inertia
-        ixx="0.0190754872818101"
-        ixy="3.73759302398911E-05"
-        ixz="-0.00248411704514181"
-        iyy="0.0131348205778546"
-        iyz="1.14470662431302E-05"
-        izz="0.0247584674534283" />
+        xyz="-0.020323640474839 -0.00503417361392195 0.055304484686837"
+        rpy="0 0 0" />
+      <mass
+        value="1.72426257072843" />
+      <inertia
+        ixx="0.0201147961188581"
+        ixy="4.24552853817101E-05"
+        ixz="-0.00247781037487344"
+        iyy="0.014189694142188"
+        iyz="1.13869699220195E-05"
+        izz="0.0268274687148955" />
     </inertial>
     <visual>
@@ -29,5 +28,5 @@
         name="">
         <color
-          rgba="0.717647058823529 0.976470588235294 1 1" />
+          rgba="0.792156862745098 0.819607843137255 0.933333333333333 1" />
       </material>
     </visual>
@@ -42,4 +41,5 @@
     </collision>
   </link>
+  <link name="base_footprint"></link>
   <joint name="base_joint" type="fixed">
     <parent link="base_footprint"/>
@@ -48,18 +48,71 @@
   </joint>
   <link
+    name="WL_Link">
+    <inertial>
+      <origin
+        xyz="-3.89171393028187E-10 -0.013931690521404 1.86314953048994E-10"
+        rpy="0 0 0" />
+      <mass
+        value="0.0333822790515451" />
+      <inertia
+        ixx="1.51686308540204E-05"
+        ixy="9.58150429074449E-17"
+        ixz="-1.67624352726415E-13"
+        iyy="2.57516582391557E-05"
+        iyz="-2.86237051388777E-15"
+        izz="1.5168630582853E-05" />
+    </inertial>
+    <visual>
+      <origin
+        xyz="0 0 0"
+        rpy="0 0 0" />
+      <geometry>
+        <mesh
+          filename="package://robot_description/meshes/WL_Link.STL" />
+      </geometry>
+      <material
+        name="">
+        <color
+          rgba="0 0.717647058823529 0.968627450980392 1" />
+      </material>
+    </visual>
+    <collision>
+      <origin
+        xyz="0 0 0"
+        rpy="0 0 0" />
+      <geometry>
+        <mesh
+          filename="package://robot_description/meshes/WL_Link.STL" />
+      </geometry>
+    </collision>
+  </link>
+  <joint
+    name="WL"
+    type="continuous">
+    <origin
+      xyz="0.015798 -0.10986 -0.03"
+      rpy="0 0 0" />
+    <parent
+      link="base_link" />
+    <child
+      link="WL_Link" />
+    <axis
+      xyz="0 1 0" />
+  </joint>
+  <link
     name="WR_Link">
     <inertial>
       <origin
-        xyz="2.17257403040128E-10 3.43708117522823E-11 -6.24044298874749E-10"
-        rpy="0 0 0" />
-      <mass
-        value="0.0218252247010597" />
-      <inertia
-        ixx="1.17812000776056E-05"
-        ixy="2.65132424286343E-15"
-        ixz="-1.33187854369566E-13"
-        iyy="2.00954687846381E-05"
-        iyz="2.48038040702484E-16"
-        izz="1.17812004135953E-05" />
+        xyz="1.41898146011066E-10 0.0139316905214036 -4.07469818303197E-10"
+        rpy="0 0 0" />
+      <mass
+        value="0.0333822790515455" />
+      <inertia
+        ixx="1.51686305491668E-05"
+        ixy="2.83393695898371E-15"
+        ixz="-1.33523495785501E-13"
+        iyy="2.57516582391559E-05"
+        iyz="-4.13340954267257E-16"
+        izz="1.51686308877069E-05" />
     </inertial>
     <visual>
@@ -74,5 +127,5 @@
         name="">
         <color
-          rgba="0.333333333333333 0.333333333333333 0.333333333333333 1" />
+          rgba="0 0.717647058823529 0.968627450980392 1" />
       </material>
     </visual>
@@ -91,5 +144,5 @@
     type="continuous">
     <origin
-      xyz="0.0177301648510787 0.131206101652453 -0.0177932693139423"
+      xyz="0.015798 0.10986 -0.03"
       rpy="0 0 0" />
     <parent
@@ -101,71 +154,18 @@
   </joint>
   <link
-    name="WL_Link">
-    <inertial>
-      <origin
-        xyz="2.17257642431967E-10 -3.43708117522823E-11 6.24044347447006E-10"
-        rpy="0 0 0" />
-      <mass
-        value="0.0218252247010597" />
-      <inertia
-        ixx="1.17812000776056E-05"
-        ixy="-2.65138193063355E-15"
-        ixz="1.33187821490352E-13"
-        iyy="2.00954687846381E-05"
-        iyz="2.47965600798296E-16"
-        izz="1.17812004135952E-05" />
-    </inertial>
-    <visual>
-      <origin
-        xyz="0 0 0"
-        rpy="0 0 0" />
-      <geometry>
-        <mesh
-          filename="package://robot_description/meshes/WL_Link.STL" />
-      </geometry>
-      <material
-        name="">
-        <color
-          rgba="0.333333333333333 0.333333333333333 0.333333333333333 1" />
-      </material>
-    </visual>
-    <collision>
-      <origin
-        xyz="0 0 0"
-        rpy="0 0 0" />
-      <geometry>
-        <mesh
-          filename="package://robot_description/meshes/WL_Link.STL" />
-      </geometry>
-    </collision>
-  </link>
-  <joint
-    name="WL"
-    type="continuous">
-    <origin
-      xyz="0.0177301648510796 -0.145293898347547 -0.0177932693139432"
-      rpy="0 0 0" />
-    <parent
-      link="base_link" />
-    <child
-      link="WL_Link" />
-    <axis
-      xyz="0 -1 0" />
-  </joint>
-  <link
     name="SF_Link">
     <inertial>
       <origin
-        xyz="-0.000805650652548284 -0.0100000000000169 -4.48165838483339E-06"
-        rpy="0 0 0" />
-      <mass
-        value="0.0386238363179237" />
-      <inertia
-        ixx="7.66294109641648E-06"
-        ixy="-3.87614098918062E-20"
-        ixz="-2.4288962364226E-11"
-        iyy="1.29044379500025E-05"
-        iyz="4.98926346371039E-24"
-        izz="7.66293122817673E-06" />
+        xyz="-0.00109034149189896 0.00021801111856061 0.000402219794071071"
+        rpy="0 0 0" />
+      <mass
+        value="0.0452273710021345" />
+      <inertia
+        ixx="1.01682869627524E-05"
+        ixy="-2.36291185766769E-11"
+        ixz="-5.31435802143934E-20"
+        iyy="1.01682729665126E-05"
+        iyz="-1.00868790747467E-21"
+        izz="1.74874180521558E-05" />
     </inertial>
     <visual>
@@ -197,6 +197,6 @@
     type="fixed">
     <origin
-      xyz="0.147657245661737 -0.00230926178691363 -0.0281473490716644"
-      rpy="0 0 0" />
+      xyz="0.13766 -0.0050587 -0.036634"
+      rpy="1.5708 0 0" />
     <parent
       link="base_link" />
@@ -204,5 +204,5 @@
       link="SF_Link" />
     <axis
-      xyz="0 0 0" />
+      xyz="0 0 1" />
   </joint>
   <link
@@ -210,15 +210,15 @@
     <inertial>
       <origin
-        xyz="-0.000805650652548243 -0.010000000000016 -4.48165838390358E-06"
-        rpy="0 0 0" />
-      <mass
-        value="0.0386238363179237" />
-      <inertia
-        ixx="7.66294109641648E-06"
-        ixy="-3.68375268562799E-20"
-        ixz="-2.42889623642261E-11"
-        iyy="1.29044379500025E-05"
-        iyz="1.58181461119993E-21"
-        izz="7.66293122817673E-06" />
+        xyz="-0.000802433467456828 4.71434097780443E-07 5.98745066350782E-05"
+        rpy="0 0 0" />
+      <mass
+        value="0.0418627718069573" />
+      <inertia
+        ixx="8.84835409421031E-06"
+        ixy="-2.38448429704364E-11"
+        ixz="2.57290383529941E-22"
+        iyy="8.84834113064509E-06"
+        iyz="1.00437728269628E-21"
+        izz="1.50655958892102E-05" />
     </inertial>
     <visual>
@@ -250,118 +250,70 @@
     type="fixed">
     <origin
-      xyz="-0.112342754338263 -0.00230926178691549 -0.0281473490716663"
+      xyz="-0.10234 -0.0050587 -0.036634"
+      rpy="1.5708 0 0" />
+    <parent
+      link="base_link" />
+    <child
+      link="SB_Link" />
+    <axis
+      xyz="0 0 1" />
+  </joint>
+  <link
+    name="Camera_Link">
+    <inertial>
+      <origin
+        xyz="-0.00770923724752959 -2.63339267868729E-05 0.000162555472316084"
+        rpy="0 0 0" />
+      <mass
+        value="0.00154848047913568" />
+      <inertia
+        ixx="9.81432463144103E-08"
+        ixy="-1.55039476124509E-11"
+        ixz="-2.74782275446747E-09"
+        iyy="6.1527176704902E-08"
+        iyz="3.76746360401982E-10"
+        izz="5.63298191001056E-08" />
+    </inertial>
+    <visual>
+      <origin
+        xyz="0 0 0"
+        rpy="0 0 0" />
+      <geometry>
+        <mesh
+          filename="package://robot_description/meshes/Camera_Link.STL" />
+      </geometry>
+      <material
+        name="">
+        <color
+          rgba="0.792156862745098 0.819607843137255 0.933333333333333 1" />
+      </material>
+    </visual>
+    <collision>
+      <origin
+        xyz="0 0 0"
+        rpy="0 0 0" />
+      <geometry>
+        <mesh
+          filename="package://robot_description/meshes/Camera_Link.STL" />
+      </geometry>
+    </collision>
+  </link>
+  <joint
+    name="Camera"
+    type="fixed">
+    <origin
+      xyz="0.1752 -0.0080928 0.068362"
       rpy="0 0 0" />
     <parent
       link="base_link" />
     <child
-      link="SB_Link" />
-    <axis
-      xyz="0 0 0" />
-  </joint>
-  <link
-    name="LD_Link">
-    <inertial>
-      <origin
-        xyz="-0.00578422640618168 -0.00125205275038996 0.00393830684198931"
-        rpy="0 0 0" />
-      <mass
-        value="0.142993542442054" />
-      <inertia
-        ixx="4.62765685052203E-05"
-        ixy="-8.53448313380911E-07"
-        ixz="-3.62169352403894E-06"
-        iyy="7.3474069260353E-05"
-        iyz="2.04313263832231E-07"
-        izz="0.000107959525263795" />
-    </inertial>
-    <visual>
-      <origin
-        xyz="0 0 0"
-        rpy="0 0 0" />
-      <geometry>
-        <mesh
-          filename="package://robot_description/meshes/LD_Link.STL" />
-      </geometry>
-      <material
-        name="">
-        <color
-          rgba="0.792156862745098 0.819607843137255 0.933333333333333 1" />
-      </material>
-    </visual>
-    <collision>
-      <origin
-        xyz="0 0 0"
-        rpy="0 0 0" />
-      <geometry>
-        <mesh
-          filename="package://robot_description/meshes/LD_Link.STL" />
-      </geometry>
-    </collision>
-  </link>
-  <joint
-    name="LD"
-    type="fixed">
-    <origin
-      xyz="0.0513960422196195 0 0.1479"
-      rpy="0 0 0" />
-    <parent
-      link="base_link" />
-    <child
-      link="LD_Link" />
-    <axis
-      xyz="0 0 0" />
-  </joint>
-  <link
-    name="Camera_Link">
-    <inertial>
-      <origin
-        xyz="-0.00347923724752958 -2.63339268585291E-05 0.000162555472316084"
-        rpy="0 0 0" />
-      <mass
-        value="0.00154848047913567" />
-      <inertia
-        ixx="9.81432463144098E-08"
-        ixy="-1.55039476125308E-11"
-        ixz="-2.74782275446738E-09"
-        iyy="6.15271767049016E-08"
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
File: robot_description/urdf/robot_gazebo.xacro (robot description, xacro)
@@ -1,4 +1,4 @@
 <?xml version="1.0"?>
-<robot name="robotTRUNG" xmlns:xacro="http://ros.org/wiki/xacro">
+<robot name="alphabot" xmlns:xacro="http://ros.org/wiki/xacro">
   <transmission name="wheel_right_transmission">
     <plugin>transmission_interface/SimpleTransmission</plugin>
@@ -18,25 +18,25 @@
   <gazebo reference="WL">
     <material>Gazebo/Blue</material>
-    <mu1>2.0</mu1>
-    <mu2>2.0</mu2>
-    <kp>10000.0</kp>
+    <mu1>1000000000000000.0</mu1>
+    <mu2>1000000000000000.0</mu2>
+    <kp>1000000000000.0</kp>
     <kd>10.0</kd>
     <minDepth>0.001</minDepth>
     <maxVel>0.1</maxVel>
-    <fdir1>1 0 0</fdir1>
+    <!-- <fdir1>1 0 0</fdir1> -->
   </gazebo>
   <gazebo reference="WR">
     <material>Gazebo/Blue</material>
-    <mu1>2.0</mu1>
-    <mu2>2.0</mu2>
-    <kp>10000.0</kp>
+    <mu1>1000000000000000.0</mu1>
+    <mu2>1000000000000000.0</mu2>
+    <kp>1000000000000.0</kp>
     <kd>10.0</kd>
     <minDepth>0.001</minDepth>
     <maxVel>0.1</maxVel>
-    <fdir1>1 0 0</fdir1>
+    <!-- <fdir1>1 0 0</fdir1> -->
   </gazebo>
   <!-- Caster Wheels -->
   <gazebo reference="SB">
-    <material>Gazebo/FlatBlack</material>
+    <material>Gazebo/Blue</material>
     <mu1>0.1</mu1>
     <mu2>0.1</mu2>
@@ -47,5 +47,5 @@
   </gazebo>
   <gazebo reference="SF">
-    <material>Gazebo/FlatBlack</material>
+    <material>Gazebo/Blue</material>
     <mu1>0.1</mu1>
     <mu2>0.1</mu2>

File: robot_description/urdf/robot_ros2_control.xacro (robot description, xacro)
@@ -1,4 +1,4 @@
 <?xml version="1.0"?>
-<robot xmlns:xacro="http://www.ros.org/wiki/xacro" name="robotTRUNG">
+<robot xmlns:xacro="http://www.ros.org/wiki/xacro" name="alphabot">
     <transmission name="right_wheel_trans">
         <type>transmission_interface/SimpleTransmission</type>
