Commit message: feat: Add robot firmware and recognition packages with serial communication and YOLOv8 integration

File: robot_description/urdf/robot.urdf.xacro (robot description, xacro)
@@ -1,7 +1,221 @@
 <?xml version="1.0"?>
-<robot name ="alphabot" xmlns:xacro="http://ros.org/wiki/xacro" >
-    <xacro:arg name="is_sim" default="true"/>
-    <xacro:include filename="robot_core.xacro" />
-    <xacro:include filename="robot_ros2_control.xacro" />
-    <xacro:include filename="robot_gazebo.xacro" />
+<robot name="alphabot" xmlns:xacro="http://ros.org/wiki/xacro">
+  <!-- Start GZ or Ignition depending on ROS 2 Version -->
+  <xacro:arg name="is_ignition" default="false"/>
+  <!-- Load Simulated or Real Hardware Interfaces -->
+  <xacro:arg name="is_sim" default="true"/>
+  <!-- Include Gazebo Parameters -->
+  <xacro:include filename="$(find robot_description)/urdf/robot_gazebo.xacro" />
+  <!-- Include ros2_control Plugins -->
+  <xacro:include filename="$(find robot_description)/urdf/robot_ros2_control.xacro" />
+  <xacro:include filename="$(find robot_description)/urdf/camera.urdf.xacro" />
+  <link name="base_footprint"/>
+  <link name="base_link">
+    <inertial>
+      <origin xyz="0 0 0.04" rpy="0.0 0.25 0.3" />
+      <mass value="8.2573504e-01"/>
+      <inertia ixx="2.2124416e-02" ixy="-1.2294101e-04" ixz="3.4938785e-04"
+               iyy="2.1193702e-02" iyz="-5.0120904e-05"
+               izz="2.0064271e-02" />
+    </inertial>
+    <visual>
+      <origin xyz="0 0 0" rpy="0 0 0" />
+      <geometry>
+        <mesh filename="package://robot_description/meshes/base_link.STL" />
+      </geometry>
+      <material name="black"/>
+    </visual>
+    <collision>
+      <origin xyz="0 0 0" rpy="0 0 0" />
+      <geometry>
+        <mesh filename="package://robot_description/meshes/base_link.STL" />
+      </geometry>
+    </collision>
+  </link>
+  <joint name="base_joint" type="fixed">
+    <parent link="base_footprint"/>
+    <child link="base_link" />
+    <origin xyz="0 0 0.033" rpy="0 0 0"/>
+  </joint>
+  <link name="wheel_right_link">
+    <inertial>
+      <origin xyz="0 -0.014 0" rpy="0 0 0" />
+      <mass value="0.0530086090966721" />
+      <inertia ixx="1.88176298336665E-05" ixy="-4.8444933029987E-10" ixz="1.88163708851143E-08"
+               iyy="3.11510738647764E-05" iyz="-6.93560663069607E-11"
+               izz="1.8801969558182E-05" />
+    </inertial>
+    <visual>
+      <origin xyz="0 0 0" rpy="1.57 0 0" />
+      <geometry>
+        <mesh filename="package://robot_description/meshes/wheel_right_link.STL" />
+      </geometry>
+      <material name="blue"/>
+    </visual>
+    <collision>
+      <origin xyz="0 -0.015 0" rpy="1.57 0 0" />
+      <geometry>
+        <sphere radius="0.033"/>
+      </geometry>
+    </collision>
+  </link>
+  <joint name="wheel_right_joint" type="continuous">
+    <origin xyz="0 -0.0701101849418637 0" rpy="0 0 0" />
+    <parent link="base_link" />
+    <child link="wheel_right_link" />
+    <axis xyz="0 1 0" />
+  </joint>
+  <link
+    name="wheel_left_link">
+    <inertial>
+      <origin xyz="0 0.014 0" rpy="0 0 0" />
+      <mass value="0.0530086043217644" />
+      <inertia ixx="1.8792911368909E-05"  ixy="3.31256392204584E-10" ixz="-1.14082001662767E-08"
+               iyy="3.11510738759073E-05" iyz="-3.60499245082192E-10"
+               izz="1.88266886146847E-05" />
+    </inertial>
+    <visual>
+      <origin xyz="0 0 0" rpy="-1.57 0 0" />
+      <geometry>
+        <mesh filename="package://robot_description/meshes/wheel_left_link.STL" />
+      </geometry>
+      <material name="blue"/>
+    </visual>
+    <collision>
+      <origin xyz="0 0.015 0" rpy="-1.57 0 0" />
+      <geometry>
+        <sphere radius="0.033"/>
+      </geometry>
+    </collision>
+  </link>
+  <joint name="wheel_left_joint" type="continuous">
+    <origin xyz="0 0.0701101849418642 0" rpy="0 0 0" />
+    <parent link="base_link" />
+    <child link="wheel_left_link" />
+    <axis xyz="0 1 0" />
+  </joint>
+  <link name="caster_front_link">
+    <inertial>
+      <origin xyz="3.89968128948481E-07 2.40073004698083E-07 0.00219173397061506" rpy="0 0 0" />
+      <mass value="1.44379265037903E-06" />
+      <inertia ixx="7.23075276010246E-11" ixy="-6.10956883467859E-16" ixz="2.22849693525031E-15"
+               iyy="3.8713793085917E-11"  iyz="2.93909858781952E-15"
+               izz="1.00967486676306E-10" />
+    </inertial>
+    <visual>
+      <origin xyz="0 0 0" rpy="0 0 0" />
+      <geometry>
+        <mesh filename="package://robot_description/meshes/caster_front_link.STL" />
+      </geometry>
+      <material name="silver"/>
+    </visual>
+    <collision>
+      <origin xyz="0 0 0" rpy="0 0 0" />
+      <geometry>
+        <sphere radius="0.005"/>
+      </geometry>
+    </collision>
+  </link>
+  <joint name="caster_front_joint" type="fixed">
+    <origin xyz="0.04755 0 -0.0275" rpy="0 0 0" />
+    <parent link="base_link" />
+    <child link="caster_front_link" />
+    <axis xyz="0 0 0" />
+  </joint>
+  <link name="caster_rear_link">
+    <inertial>
+      <origin xyz="3.8996812895542E-07 2.40073004698083E-07 0.00219173397061509" rpy="0 0 0" />
+      <mass value="1.44379265037902E-06" />
+      <inertia ixx="7.23075276010246E-11" ixy="-6.10956872363424E-16" ixz="2.22849693527207E-15"
+               iyy="3.87137930859167E-11" iyz="2.939098587861E-15"
+               izz="1.00967486676306E-10" />
+    </inertial>
+    <visual>
+      <origin xyz="0 0 0" rpy="0 0 0" />
+      <geometry>
+        <mesh filename="package://robot_description/meshes/caster_rear_link.STL" />
+      </geometry>
+      <material name="silver"/>
+    </visual>
+    <collision>
+      <origin xyz="0 0 0" rpy="0 0 0" />
+      <geometry>
+        <sphere radius="0.005"/>
+      </geometry>
+    </collision>
+  </link>
+  <joint name="caster_rear_joint" type="fixed">
+    <origin xyz="-0.04755 0 -0.0275" rpy="0 0 0" />
+    <parent link="base_link" />
+    <child link="caster_rear_link" />
+    <axis xyz="0 0 0" />
+  </joint>
+  <link name="imu_link">
+    <inertial>
+      <origin xyz="-0.00552433659106688 0.000168210391520346 0.000514000497342681" rpy="0 0 0" />
+      <mass value="0.000528415362211671" />
+      <inertia ixx="1.46176048428261E-08" ixy="1.40015117949421E-10" ixz="-1.99633872937403E-12"
+               iyy="8.59662482954888E-09" iyz="7.52375112767959E-12"
+               izz="2.30279421279312E-08" />
+    </inertial>
+    <visual>
+      <origin xyz="0 0 0" rpy="0 0 0" />
+      <geometry>
+        <mesh filename="package://robot_description/meshes/imu_link.STL" />
+      </geometry>
+      <material name="blue"/>
+    </visual>
+    <collision>
+      <origin xyz="0 0 0" rpy="0 0 0" />
+      <geometry>
+        <mesh filename="package://robot_description/meshes/imu_link.STL" />
+      </geometry>
+    </collision>
+  </link>
+  <joint name="imu_joint" type="fixed">
+    <origin xyz="0 0 0.0698986241758014" rpy="0 0 0" />
+    <parent link="base_link" />
+    <child link="imu_link" />
+    <axis xyz="0 0 0" />
+  </joint>
+  <link name="laser_link">
+    <inertial>
+      <origin xyz="-0.011945780406062 -0.000381929217680526 -0.0170649378129477" rpy="0 0 0" />
+      <mass value="0.073084435549317" />
+      <inertia ixx="1.96074931730795E-05" ixy="-3.62091076640009E-07" ixz="4.28230084046735E-07"
+               iyy="2.40983835136327E-05" iyz="1.50180909250652E-08"
+               izz="4.14184164228595E-05" />
+    </inertial>
+    <visual>
+      <origin xyz="0 0 0" rpy="0 0 0" />
+      <geometry>
+        <mesh filename="package://robot_description/meshes/laser_link.STL" />
+      </geometry>
+      <material name="dark_grey"/>
+    </visual>
+    <collision>
+      <origin xyz="0 0 0" rpy="0 0 0" />
+      <geometry>
+        <mesh filename="package://robot_description/meshes/laser_link.STL" />
+      </geometry>
+    </collision>
+  </link>
+  <joint name="laser_joint" type="fixed">
+    <origin xyz="-0.0050526 -0.0023221 0.1208" rpy="0 0 3.14" />
+    <parent link="base_link" />
+    <child link="laser_link" />
+    <axis xyz="0 0 0" />
+  </joint>
+  <material name="blue">
+    <color rgba="0 0 1 1"/>
+  </material>
+  <material name="black">
+    <color rgba="0 0 0 1"/>
+  </material>
+  <material name="silver">
+    <color rgba="0.79 0.82 0.93 1"/>
+  </material>
+  <material name="dark_grey">
+    <color rgba="0.3 0.3 0.3 1"/>
+  </material>
 </robot>

File: robot_description/urdf/robot_gazebo.xacro (robot description, xacro)
@@ -4,5 +4,5 @@
     <plugin>transmission_interface/SimpleTransmission</plugin>
     <actuator name="wheel_right_motor" role="actuator_right"/>
-    <joint name="WR"    role="joint_right">
+    <joint name="wheel_right_joint"    role="joint_right">
       <mechanical_reduction>1.0</mechanical_reduction>
     </joint>
@@ -11,10 +11,10 @@
     <plugin>transmission_interface/SimpleTransmission</plugin>
     <actuator name="wheel_left_motor" role="actuator_left"/>
-    <joint name="WL"    role="joint_left">
+    <joint name="wheel_left_joint"    role="joint_left">
       <mechanical_reduction>1.0</mechanical_reduction>
     </joint>
   </transmission>
   <!-- Wheels -->
-  <gazebo reference="WL">
+  <gazebo reference="wheel_left_link">
     <material>Gazebo/Blue</material>
     <mu1>1000000000000000.0</mu1>
@@ -26,5 +26,5 @@
     <!-- <fdir1>1 0 0</fdir1> -->
   </gazebo>
-  <gazebo reference="WR">
+  <gazebo reference="wheel_right_link">
     <material>Gazebo/Blue</material>
     <mu1>1000000000000000.0</mu1>
@@ -37,6 +37,5 @@
   </gazebo>
   <!-- Caster Wheels -->
-  <gazebo reference="SB">
-    <material>Gazebo/Blue</material>
+  <gazebo reference="caster_rear_link">
     <mu1>0.1</mu1>
     <mu2>0.1</mu2>
@@ -46,6 +45,5 @@
     <maxVel>1.0</maxVel>
   </gazebo>
-  <gazebo reference="SF">
-    <material>Gazebo/Blue</material>
+  <gazebo reference="caster_front_link">
     <mu1>0.1</mu1>
     <mu2>0.1</mu2>
@@ -64,5 +62,5 @@
   </gazebo>
   <!-- IMU -->
-  <gazebo reference="IMU_Link">
+  <gazebo reference="imu_link">
     <sensor name="imu" type="imu">
         <always_on>true</always_on>
@@ -86,5 +84,5 @@
                 <mean>0.0</mean>
                 <stddev>2e-4</stddev>
-              </noise>
+              </noise>wheel_left_link
             </z>
           </angular_velocity>
@@ -114,5 +112,5 @@
   </gazebo>
   <!-- 2D Laser Sensor -->
-  <gazebo reference="LD_Link">
+  <gazebo reference="laser_link">
     <sensor name="lidar" type="ray">
       <always_on>true</always_on>
@@ -144,9 +142,9 @@
         </ros>
         <output_type>sensor_msgs/LaserScan</output_type>
-        <frame_name>LD_Link</frame_name>
+        <frame_name>laser_link</frame_name>
       </plugin>
     </sensor>
   </gazebo>
-  <gazebo reference="Camera_Link">
+  <!-- <gazebo reference="Camera_Link">
     <sensor name="camera" type="camera">
       <update_rate>30.0</update_rate>
@@ -171,3 +169,4 @@
     </sensor>
   </gazebo>
+   -->
 </robot>

File: robot_description/urdf/robot_ros2_control.xacro (robot description, xacro)
@@ -3,5 +3,5 @@
     <transmission name="right_wheel_trans">
         <type>transmission_interface/SimpleTransmission</type>
-        <joint name="WR">
+        <joint name="wheel_right_joint">
             <hardwareInterface>hardware_interface::HW_IF_VELOCITY</hardwareInterface>
         </joint>
@@ -13,5 +13,5 @@
     <transmission name="left_wheel_trans">
         <type>transmission_interface/SimpleTransmission</type>
-        <joint name="WL">
+        <joint name="wheel_left_joint">
             <hardwareInterface>hardware_interface::HW_IF_VELOCITY</hardwareInterface>
         </joint>
@@ -31,9 +31,9 @@
             <hardware>
                 <plugin>robot_firmware/RobotInterface</plugin>
-                <param name="port">/dev/arduino_uno</param>
+                <param name="port">/dev/ttyUSB0</param>
             </hardware>
         </xacro:unless>
             <!-- ros2_control Common Interfaces -->
-        <joint name="WR">
+        <joint name="wheel_right_joint">
             <command_interface name="velocity">
             <param name="min">-5</param>
@@ -43,5 +43,5 @@
             <state_interface name="velocity" />
         </joint>
-        <joint name="WL">
+        <joint name="wheel_left_joint">
             <command_interface name="velocity">
             <param name="min">-5</param>
